Commit message: Scaling  to 1 the urdf models for collision workaround. Handling linear collisions between static objects and moving shapes.

File: data/urdf/blade.urdf (robot description, URDF)
Before this commit: robot blade, 1 links, 0 joints
Links:
- link body: geometry collision mesh filename=blade.obj scale=1.0 1.0 1.0; visual mesh filename=blade.obj scale=1.0 1.0 1.0

File: data/urdf/cylinder.urdf (robot description, URDF)
Before this commit: robot cylinder, 1 links, 0 joints
Links:
- link body: geometry collision mesh filename=cylinder.obj scale=1.0 1.0 1.0; visual mesh filename=cylinder.obj scale=1.0 1.0 1.0
