Commit message: finalized regression test

File: data/urdf/test/issue838.urdf (robot description, URDF)
Before this commit: robot issue838, 5 links, 4 joints
Links:
- removed link arm_0
- removed link arm_1
- removed link arm_2
- removed link arm_base
- removed link base_link
- added link link_0, mass 10.0; visual box size=1 1 1; visual box size=1 1 1
- added link link_1; visual box size=1 1 1; visual box size=1 1 1
- added link link_2, mass 0.855; visual box size=1 1 1; visual box size=1 1 1
Joints:
- removed joint arm_0_1
- removed joint arm_1_2
- removed joint arm_base_arm_0
- removed joint base_link_arm_base
- added joint 0_to_1: type fixed, parent link_0, child link_1, origin xyz=0 0 0 rpy=0 0 0
- added joint 1_to_2: type revolute, parent link_1, child link_2, origin xyz=0 0 0 rpy=0 0 0, axis 0 0 1, limit lower=-3.14159265359 upper=3.14159265359 effort=2.5 velocity=3.00545697193
