Commit message: Testing minitaur with closed loops

File: data/urdf/minitaur/minitaur.urdf (robot description, URDF)
Before this commit: robot quadruped, 27 links, 26 joints
Joints:
- joint chassis_left_center: origin xyz=0.0 0.10 0.0 rpy=0.0872665 0 0 -> xyz=0.0 0.10 0.0 rpy=0.0 0 0
- joint chassis_right_center: origin xyz=0.0 -0.10 0.0 rpy=-0.0872665 0 0 -> xyz=0.0 -0.10 0.0 rpy=-0.0 0 0
- joint knee_back_leftL_link: origin xyz=0.0 0.01 .055 rpy=0 0 0 -> xyz=0.0 0.00 .055 rpy=0 0 0
- joint knee_back_leftR_link: origin xyz=0.0 0.01 .055 rpy=0 0 0 -> xyz=0.0 0.00 .055 rpy=0 0 0
- joint knee_back_rightL_link: origin xyz=0.0 0.01 .055 rpy=0 0 0 -> xyz=0.0 0.00 .055 rpy=0 0 0
- joint knee_back_rightR_link: origin xyz=0.0 0.01 .055 rpy=0 0 0 -> xyz=0.0 0.00 .055 rpy=0 0 0
- joint knee_front_leftL_link: origin xyz=0.0 0.01 .055 rpy=0 0 0 -> xyz=0.0 0.00 .055 rpy=0 0 0
- joint knee_front_leftR_link: origin xyz=0.0 0.01 .055 rpy=0 0 0 -> xyz=0.0 0.00 .055 rpy=0 0 0
- joint knee_front_rightL_link: origin xyz=0.0 0.01 .055 rpy=0 0 0 -> xyz=0.0 0.00 .055 rpy=0 0 0
- joint knee_front_rightR_link: origin xyz=0.0 0.01 .055 rpy=0 0 0 -> xyz=0.0 0.00 .055 rpy=0 0 0
