Commit message: Revert to the default joint limits of the Barrett WAM arm

File: data/urdf/wam/wam.urdf (robot description, URDF)
Before this commit: robot wam, 9 links, 8 joints
Joints:
- joint /j1: limit lower=0.54159265359 upper=5.74159265359 effort=1.8 velocity=0.75 -> lower=-2.6 upper=2.6 effort=1.8 velocity=0.75
