Commit message: Attribute the Atlas sample and keep only WAM's BSD files (#3882)

File: data/urdf/wam/wam.urdf (robot description, URDF)
Before this commit: robot wam, 9 links, 8 joints
Links:
- link /wam1: geometry collision mesh filename=package://herb_description/meshes/wam/wam1_collision.STL; visual mesh filename=package://herb_description/meshes/wam/wam1.STL
- link /wam2: geometry collision mesh filename=package://herb_description/meshes/wam/wam2_collision.STL; visual mesh filename=package://herb_description/meshes/wam/wam2.STL
- link /wam3: geometry collision mesh filename=package://herb_description/meshes/wam/wam3_collision.STL; visual mesh filename=package://herb_description/meshes/wam/wam3.STL
- link /wam4: geometry collision mesh filename=package://herb_description/meshes/wam/wam4_collision.STL; visual mesh filename=package://herb_description/meshes/wam/wam4.STL
- link /wam5: geometry collision mesh filename=package://herb_description/meshes/wam/wam5_collision.STL; visual mesh filename=package://herb_description/meshes/wam/wam5.STL
- link /wam6: geometry collision mesh filename=package://herb_description/meshes/wam/wam6_collision.STL; visual mesh filename=package://herb_description/meshes/wam/wam6.STL
- link /wam7: geometry collision mesh filename=package://herb_description/meshes/wam/wam7_collision.STL; visual mesh filename=package://herb_description/meshes/wam/wam7.STL
- link /wam_base: geometry collision mesh filename=package://herb_description/meshes/wam/wam_base_collision.STL; visual mesh filename=package://herb_description/meshes/wam/wam_base.STL
